File: PSU/PCB-Rev.1/psu-pcb/psu-pcb.sch (KiCad schematic (older format))
At the start: 60 parts, among them J1 Conn_02x07_Odd_Even, J2 OSTTC022162, J3 OSTTC022162, J4 OSTTC022162, J5 OSTTC022162, J6 OSTTC022162, J7 OSTTC022162, J8 Conn_02x05_Odd_Even, Q1 FQP27P06, Q2 2N7002, Q3 2N7002, Q4 2N7002, Q5 2N7002, U1 PIC12F1501-IP, U2 ADS1110

Commit message: Poseidon PSU pcb
Parts:
- C1, C6: footprint (none) -> Capacitor_SMD:C_0805_2012Metric
- C10: renamed from C13; footprint (none) -> Capacitor_THT:CP_Radial_D7.5mm_P2.50mm
- C11: renamed from C8; footprint (none) -> Capacitor_THT:CP_Radial_D7.5mm_P2.50mm
- C12: renamed from C9; footprint (none) -> Capacitor_THT:CP_Radial_D7.5mm_P2.50mm
- C2, C3, C5, C7: footprint (none) -> Capacitor_THT:CP_Radial_D7.5mm_P2.50mm
- C4: renamed from C11; footprint (none) -> Capacitor_THT:CP_Radial_D7.5mm_P2.50mm
- C8: renamed from C12; footprint (none) -> Capacitor_THT:CP_Radial_D7.5mm_P2.50mm
- C9: renamed from C10; footprint (none) -> Capacitor_THT:CP_Radial_D7.5mm_P2.50mm
- J1: footprint (none) -> Connector_IDC:IDC-Header_2x07_P2.54mm_Vertical_Lock
- J8: footprint (none) -> Connector_IDC:IDC-Header_2x05_P2.54mm_Vertical
- R1, R17, R2, R3, R4, R5, R6, R7, R8, R9: footprint (none) -> Resistor_SMD:R_0805_2012Metric
- R10: renamed from R18; footprint (none) -> Resistor_SMD:R_0805_2012Metric
- R11: renamed from R12; footprint (none) -> Resistor_SMD:R_0805_2012Metric
- R12: renamed from R14; footprint (none) -> Resistor_SMD:R_0805_2012Metric
- R13: renamed from R16; footprint (none) -> Resistor_SMD:R_0805_2012Metric
- R14: renamed from R10; footprint (none) -> Resistor_SMD:R_0805_2012Metric
- R15: renamed from R11; footprint (none) -> Resistor_SMD:R_0805_2012Metric
- R16: renamed from R13; footprint (none) -> Resistor_SMD:R_0805_2012Metric
- R18: renamed from R15; footprint (none) -> Resistor_SMD:R_0805_2012Metric
- renumbered L4 to L2, L2 to L4, Q3 to Q1, Q4 to Q2, Q5 to Q3, Q1 to Q4, Q2 to Q5
Connections:
- net at PS2.4 (TRIM), R8.1: now also C6.1; no longer C6.2
- net at R9.2: now also C6.2; no longer C6.1
Other:
- moved on the sheet: C10, C4, C5, C6, C7, C8, C9, D4, D5, J5, L2, L3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
