File: PSU/PCB-Rev.1/psu-pcb/psu-pcb.sch (KiCad schematic (older format))
At the start: 60 parts, among them J1 Conn_02x07_Odd_Even, J2 OSTTC022162, J3 OSTTC022162, J4 OSTTC022162, J5 OSTTC022162, J6 OSTTC022162, J7 OSTTC022162, J8 Conn_02x05_Odd_Even, Q1 2N7002, Q2 2N7002, Q3 2N7002, Q4 FQP27P06, Q5 2N7002, U1 PIC12F1501-IP, U2 ADS1110

Commit message: update psu and hat
Other:
- moved on the sheet: C11, C12, L4, Q1, Q4, Q5, R11, R14, R15

Commit message: smt to TH
Parts:
- removed C6: C, Capacitor_SMD:C_0805_2012Metric, symbol Device:C
- removed J3, J4, J5, J6: OSTTC022162, digikey-footprints:Term_Block_1x2_P5.08MM, symbol psu-pcb-rescue:OSTTC022162-dk_Terminal-Blocks-Wire-to-Board
- removed J8: Conn_02x05_Odd_Even, Connector_IDC:IDC-Header_2x05_P2.54mm_Vertical, symbol Connector_Generic:Conn_02x05_Odd_Even
- removed PS2: APXW005A0X3-SRZ, APXW005A0X3SRZ, symbol psu-pcb-rescue:APXW005A0X3-SRZ-APXW005A0X3-SRZ
- removed Q1, Q2, Q3, Q5: 2N7002, digikey-footprints:SOT-23-3, symbol psu-pcb-rescue:2N7002-dk_Transistors-FETs-MOSFETs-Single
- removed R8: R_US, Resistor_SMD:R_0805_2012Metric, symbol Device:R_US
- removed U2: ADS1110, Package_TO_SOT_SMD:SOT-23-6, symbol Analog_ADC:ADS1110
- added C13, C17: 10UF, Capacitor_THT:C_Rect_L7.0mm_W2.0mm_P5.00mm, symbol Device:C
- added C14: 4.7UF 50V, Capacitor_THT:C_Rect_L7.0mm_W2.0mm_P5.00mm, symbol Device:C
- added C15, C18: 0.1UF, Capacitor_THT:C_Rect_L7.0mm_W2.0mm_P5.00mm, symbol Device:C
- added C16: 1NF 2KV, Capacitor_THT:C_Rect_L7.0mm_W2.0mm_P5.00mm, symbol Device:C
- added J10, J11, J12, J13, J14, J15, J16, J3, J4, J5, J6, J9: Conn_01x02, Connector_JST:JST_EH_B2B-EH-A_1x02_P2.50mm_Vertical, symbol Connector_Generic:Conn_01x02
- added J8: Conn_01x05, Connector_PinHeader_2.54mm:PinHeader_1x05_P2.54mm_Vertical, symbol Connector_Generic:Conn_01x05
- added PS2: SKMW30F-05, SKMW30G-12:SKMW30G12, symbol SKMW30G-12:SKMW30G-12
- added Q1, Q2, Q3, Q5: 2N7000, Package_TO_SOT_THT:TO-92_Inline, symbol Transistor_FET:2N7000
- added U2: MCP3426-xSN, Package_SO:SOIC-8-1EP_3.9x4.9mm_P1.27mm_EP2.29x3mm, symbol Analog_ADC:MCP3426-xSN
- C1: value C -> 0.1u; footprint Capacitor_SMD:C_0805_2012Metric -> Capacitor_THT:C_Rect_L7.0mm_W2.5mm_P5.00mm
- C10: value CP1 -> 47UF 35V; footprint Capacitor_THT:CP_Radial_D7.5mm_P2.50mm -> Capacitor_THT:CP_Radial_D6.3mm_P2.50mm
- C11, C4: value CP1 -> 100UF 50V; footprint Capacitor_THT:CP_Radial_D7.5mm_P2.50mm -> Capacitor_THT:CP_Radial_D8.0mm_P5.00mm
- C12, C5: value CP1 -> 47UF 50V; footprint Capacitor_THT:CP_Radial_D7.5mm_P2.50mm -> Capacitor_THT:CP_Radial_D6.3mm_P2.50mm
- C2: value CP1 -> 10u 35v; footprint Capacitor_THT:CP_Radial_D7.5mm_P2.50mm -> Capacitor_THT:CP_Radial_D5.0mm_P2.50mm
- C3: value CP1 -> 10u 10v; footprint Capacitor_THT:CP_Radial_D7.5mm_P2.50mm -> Capacitor_THT:CP_Radial_D5.0mm_P2.50mm
- C7: value CP1 -> 330uf 16v; footprint Capacitor_THT:CP_Radial_D7.5mm_P2.50mm -> Capacitor_THT:CP_Radial_D8.0mm_P5.00mm
- C8: value CP1 -> 100UF 35V; footprint Capacitor_THT:CP_Radial_D7.5mm_P2.50mm -> Capacitor_THT:CP_Radial_D8.0mm_P5.00mm
- C9: value CP1 -> 330UF 50V; footprint Capacitor_THT:CP_Radial_D7.5mm_P2.50mm -> Capacitor_THT:CP_Radial_D10.0mm_P5.00mm
- D2, D3, D4, D5, D6: footprint digikey-footprints:0805 -> LED_THT:LED_D3.0mm_Clear
- F1, F2: footprint digikey-footprints:1206 -> Fuse:Fuse_Littelfuse_372_D8.50mm
- L1: value 13R106C -> 1uh
- L3: value 13R106C -> 2.2UH 4A
- L4: value 13R106C -> 1UH
- R1, R14, R15: value R_US -> 10k; footprint Resistor_SMD:R_0805_2012Metric -> Resistor_THT:R_Axial_DIN0207_L6.3mm_D2.5mm_P2.54mm_Vertical
- R10: value R_US -> 220; footprint Resistor_SMD:R_0805_2012Metric -> Resistor_THT:R_Axial_DIN0207_L6.3mm_D2.5mm_P2.54mm_Vertical
- R11, R12, R13: value R_US -> 1k; footprint Resistor_SMD:R_0805_2012Metric -> Resistor_THT:R_Axial_DIN0207_L6.3mm_D2.5mm_P2.54mm_Vertical
- R16: value R_US -> 2k; footprint Resistor_SMD:R_0805_2012Metric -> Resistor_THT:R_Axial_DIN0207_L6.3mm_D2.5mm_P2.54mm_Vertical
- R17: value R_US -> 560; footprint Resistor_SMD:R_0805_2012Metric -> Resistor_THT:R_Axial_DIN0207_L6.3mm_D2.5mm_P2.54mm_Vertical
- R18: value R_US -> 3.9k; footprint Resistor_SMD:R_0805_2012Metric -> Resistor_THT:R_Axial_DIN0207_L6.3mm_D2.5mm_P2.54mm_Vertical
- R2: value R_US -> 7.87k 0.1%; footprint Resistor_SMD:R_0805_2012Metric -> Resistor_THT:R_Axial_DIN0207_L6.3mm_D2.5mm_P2.54mm_Vertical
- R3: value R_US -> 1.27k 0.1%; footprint Resistor_SMD:R_0805_2012Metric -> Resistor_THT:R_Axial_DIN0207_L6.3mm_D2.5mm_P2.54mm_Vertical
- R4: value R_US -> XX; footprint Resistor_SMD:R_0805_2012Metric -> Resistor_THT:R_Axial_DIN0207_L6.3mm_D2.5mm_P2.54mm_Vertical
- R5: value R_US -> 20K; footprint Resistor_SMD:R_0805_2012Metric -> Resistor_THT:R_Axial_DIN0207_L6.3mm_D2.5mm_P2.54mm_Vertical
- R6: value R_US -> 2.87K; footprint Resistor_SMD:R_0805_2012Metric -> Resistor_THT:R_Axial_DIN0207_L6.3mm_D2.5mm_P2.54mm_Vertical
- R7: value R_US -> 24.872K; footprint Resistor_SMD:R_0805_2012Metric -> Resistor_THT:R_Axial_DIN0207_L6.3mm_D2.5mm_P2.54mm_Vertical
- R9: value R_US -> xx; footprint Resistor_SMD:R_0805_2012Metric -> Resistor_THT:R_Axial_DIN0207_L6.3mm_D2.5mm_P2.54mm_Vertical
Connections:
- net labels added: 12VOUT, 24VOUT, 3.3VOUT, 5VOUT
- wire segments 82 -> 94
Other:
- moved on the sheet: C1, C10, C4, C5, C8, C9, D4, D5, F2, L2, L3, PS1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

Commit message: update
Parts:
- PS2: symbol SKMW30G-12:SKMW30G-12 -> psu-pcb-rescue:SKMW30G-12-SKMW30G-12
Changed lines of the file:
@@
 EESchema Schematic File Version 4
-EELAYER 30 0
+LIBS:psu-pcb-cache
+EELAYER 26 0
 EELAYER END
 $Descr USLetter 11000 8500
@@
 	7300 1300 7300 1600
 $Comp
-L SKMW30G-12:SKMW30G-12 PS2
+L psu-pcb-rescue:SKMW30G-12-SKMW30G-12 PS2
 U 1 1 5E6B71D5
 P 6500 5100

Commit message: update
Parts:
- C1: value 0.1u -> 0.1UF
- C10: value 47UF 35V -> 47UF 50V
- C13, C17: value 10UF -> 10u 35v
- C15, C18: footprint Capacitor_THT:C_Rect_L7.0mm_W2.0mm_P5.00mm -> Capacitor_THT:C_Rect_L7.0mm_W2.5mm_P5.00mm
- C3: value 10u 10v -> 10u 35v
- C7: value 330uf 16v -> 330UF 50V; footprint Capacitor_THT:CP_Radial_D8.0mm_P5.00mm -> Capacitor_THT:CP_Radial_D10.0mm_P5.00mm
- C8: value 100UF 35V -> 100UF 50V
Changed lines of the file:
@@
 EESchema Schematic File Version 4
-LIBS:psu-pcb-cache
-EELAYER 26 0
+EELAYER 30 0
 EELAYER END
 $Descr USLetter 11000 8500
@@
 P 650 3350
 F 0 "C1" H 765 3396 50  0000 L CNN
-F 1 "0.1u" H 765 3305 50  0000 L CNN
+F 1 "0.1UF" H 765 3305 50  0000 L CNN
 F 2 "Capacitor_THT:C_Rect_L7.0mm_W2.5mm_P5.00mm" H 688 3200 50  0001 C CNN
 F 3 "~" H 650 3350 50  0001 C CNN
@@
 P 2150 7200
 F 0 "C3" H 2265 7246 50  0000 L CNN
-F 1 "10u 10v" H 2265 7155 50  0000 L CNN
+F 1 "10u 35v" H 2265 7155 50  0000 L CNN
 F 2 "Capacitor_THT:CP_Radial_D5.0mm_P2.50mm" H 2150 7200 50  0001 C CNN
 F 3 "~" H 2150 7200 50  0001 C CNN
@@
 P 9250 5450
 F 0 "C7" H 9365 5496 50  0000 L CNN
-F 1 "330uf 16v" H 9365 5405 50  0000 L CNN
-F 2 "Capacitor_THT:CP_Radial_D8.0mm_P5.00mm" H 9250 5450 50  0001 C CNN
+F 1 "330UF 50V" H 9365 5405 50  0000 L CNN
+F 2 "Capacitor_THT:CP_Radial_D10.0mm_P5.00mm" H 9250 5450 50  0001 C CNN
 F 3 "~" H 9250 5450 50  0001 C CNN
 	1    9250 5450
@@
 P 5050 5450
 F 0 "C8" H 5165 5496 50  0000 L CNN
-F 1 "100UF 35V" H 5165 5405 50  0000 L CNN
+F 1 "100UF 50V" H 5165 5405 50  0000 L CNN
 F 2 "Capacitor_THT:CP_Radial_D8.0mm_P5.00mm" H 5050 5450 50  0001 C CNN
 F 3 "~" H 5050 5450 50  0001 C CNN
@@
 P 5450 5450
 F 0 "C10" H 5565 5496 50  0000 L CNN
-F 1 "47UF 35V" H 5565 5405 50  0000 L CNN
+F 1 "47UF 50V" H 5565 5405 50  0000 L CNN
 F 2 "Capacitor_THT:CP_Radial_D6.3mm_P2.50mm" H 5450 5450 50  0001 C CNN
 F 3 "~" H 5450 5450 50  0001 C CNN
@@
 P 8700 5450
 F 0 "C17" H 8815 5496 50  0000 L CNN
-F 1 "10UF" H 8815 5405 50  0000 L CNN
+F 1 "10u 35v" H 8815 5405 50  0000 L CNN
 F 2 "Capacitor_THT:C_Rect_L7.0mm_W2.0mm_P5.00mm" H 8738 5300 50  0001 C CNN
 F 3 "~" H 8700 5450 50  0001 C CNN
@@
 F 0 "C18" H 9065 5496 50  0000 L CNN
 F 1 "0.1UF" H 9065 5405 50  0000 L CNN
-F 2 "Capacitor_THT:C_Rect_L7.0mm_W2.0mm_P5.00mm" H 8988 5300 50  0001 C CNN
+F 2 "Capacitor_THT:C_Rect_L7.0mm_W2.5mm_P5.00mm" H 8988 5300 50  0001 C CNN
 F 3 "~" H 8950 5450 50  0001 C CNN
 	1    8950 5450
@@
 P 5800 5450
 F 0 "C13" H 5915 5496 50  0000 L CNN
-F 1 "10UF" H 5915 5405 50  0000 L CNN
+F 1 "10u 35v" H 5915 5405 50  0000 L CNN
 F 2 "Capacitor_THT:C_Rect_L7.0mm_W2.0mm_P5.00mm" H 5838 5300 50  0001 C CNN
 F 3 "~" H 5800 5450 50  0001 C CNN
@@
 F 0 "C15" H 6315 5496 50  0000 L CNN
 F 1 "0.1UF" H 6315 5405 50  0000 L CNN
-F 2 "Capacitor_THT:C_Rect_L7.0mm_W2.0mm_P5.00mm" H 6238 5300 50  0001 C CNN
+F 2 "Capacitor_THT:C_Rect_L7.0mm_W2.5mm_P5.00mm" H 6238 5300 50  0001 C CNN
 F 3 "~" H 6200 5450 50  0001 C CNN
 	1    6200 5450
