File: Daughter-board/PCB/RPi_Hat.kicad_pcb (KiCad board)
At the start: 2 copper layers, 65 x 56.5 mm, 20 parts, among them J1 Conn_01x05, J2 RPi_GPIO, J3 Conn_01x05, J4 Conn_01x05, J5 Conn_01x07, J6 Conn_01x07, J7 Conn_01x05, J8 Conn_02x07_Odd_Even, J9 Conn_01x04, Q1 2N7002, Q2 2N7002, Q3 2N7002

Commit message: update
Parts:
- moved J3 47.6 mm to (138.4, 110.4)
- moved Q3 47.6 mm to (119.7, 114.6)
- moved J4 47.6 mm to (146.1, 110.5)
- moved J8 47.6 mm to (154.3, 90.2)
- moved ? 47.6 mm to (98.8, 121.6)
- moved ? 47.6 mm to (98.8, 72.6)
- moved G*** 47.6 mm to (114.9, 96.5)
- moved J2 47.6 mm to (127.8, 72.6)
- moved J5 47.6 mm to (139.1, 80.6)
- moved J6 47.6 mm to (139.1, 88.3)
- moved Q1 47.6 mm to (109.5, 114.7)
- moved Q2 47.6 mm to (114.6, 114.7)
- moved R1 47.6 mm to (109.6, 110.5)
- moved R3 47.6 mm to (119.7, 110.5)
- moved ? 47.6 mm to (156.8, 72.6)
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Other:
- board text added: "I2C"
- board text added: "LED"
- board text added: "PSU"
- board text added: "SPI0"
- board text added: "SPI1"
- board text added: "UART"
