File: HAT/PCB Rev.1/RPi_Hat.kicad_pcb (KiCad board)
At the start: 2 copper layers, 65 x 56.5 mm, 20 parts, among them J1 Conn_01x05, J2 RPi_GPIO, J3 Conn_01x05, J4 Conn_01x05, J5 Conn_01x07, J6 Conn_01x07, J7 Conn_01x05, J8 Conn_02x07_Odd_Even, J9 Conn_01x04, Q1 2N7000, Q2 2N7000, Q3 2N7000

Commit message: gerber files
Parts:
- ? (x4): footprint cidco:MountingHole_2.7mm_M2.5_Pad -> MountingHole:MountingHole_2.7mm_M2.5_ISO7380_Pad
Other:
- net class Default: via_dia 0.6 -> 0.8
- rule pad_to_mask_clearance: 0 -> 0.1
- rule trace_min: 0 -> 0.1524
- rule via_min_size: 0.4 -> 0.6
Changed lines of the file:
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@@
-(kicad_pcb (version 20171130) (host pcbnew 5.0.2+dfsg1-1~bpo9+1)
+(kicad_pcb (version 20171130) (host pcbnew "(5.1.5)-3")
   (general
     (thickness 1.6)
@@
   )
   (setup
-    (last_trace_width 1.27)
-    (user_trace_width 0.01)
-    (user_trace_width 0.02)
-    (user_trace_width 0.05)
-    (user_trace_width 0.1)
-    (user_trace_width 0.2)
-    (user_trace_width 0.25)
-    (user_trace_width 0.5)
-    (user_trace_width 1)
+    (last_trace_width 0.25)
+    (user_trace_width 0.635)
     (user_trace_width 1.27)
+    (user_trace_width 2.54)
+    (user_trace_width 3.81)
+    (user_trace_width 5.08)
+    (user_trace_width 6.35)
     (trace_clearance 0.2)
     (zone_clearance 0.508)
     (zone_45_only no)
-    (trace_min 0)
-    (segment_width 0.2)
-    (edge_width 0.1)
-    (via_size 0.6)
+    (trace_min 0.1524)
+    (via_size 0.8)
     (via_drill 0.4)
-    (via_min_size 0.4)
+    (via_min_size 0.6)
     (via_min_drill 0.3)
     (uvia_size 0.3)
@@
     (uvia_min_size 0.2)
     (uvia_min_drill 0.1)
+    (edge_width 0.15)
+    (segment_width 0.2)
     (pcb_text_width 0.3)
     (pcb_text_size 1.5 1.5)
@@
     (pad_size 2.75 2.75)
     (pad_drill 2.75)
-    (pad_to_mask_clearance 0)
+    (pad_to_mask_clearance 0.1)
     (solder_mask_min_width 0.25)
     (aux_axis_origin 0 0)
     (visible_elements 7FFEFFFF)
     (pcbplotparams
-      (layerselection 0x00030_80000001)
-      (usegerberextensions false)
+      (layerselection 0x010f0_ffffffff)
+      (usegerberextensions true)
       (usegerberattributes false)
       (usegerberadvancedattributes false)
@@
       (psa4output false)
       (plotreference true)
-      (plotvalue true)
+      (plotvalue false)
       (plotinvisibletext false)
-      (padsonsilk false)
+      (padsonsilk true)
       (subtractmaskfromsilk false)
       (outputformat 1)
@@
       (drillshape 0)
       (scaleselection 1)
-      (outputdirectory "meta/"))
+      (outputdirectory "gerbers/"))
   )
   (net 0 "")
@@
     (clearance 0.2)
     (trace_width 0.25)
-    (via_dia 0.6)
+    (via_dia 0.8)
     (via_drill 0.4)
     (uvia_dia 0.3)
@@
     (add_net SDA)
     (add_net TX)
+  )
+  (module MountingHole:MountingHole_2.7mm_M2.5_ISO7380_Pad (layer F.Cu)
+    (at 156.75 121.58)
+    (descr "Mounting Hole 2.7mm, M2.5, ISO7380")
+    (tags "mounting hole 2.7mm m2.5 iso7380")
+    (attr virtual)
+    (fp_text reference "" (at 0 -3.7) (layer F.SilkS)
+      (effects (font (size 1 1) (thickness 0.15)))
+    )
+    (fp_text value "" (at 0 3.7) (layer F.Fab) hide
+      (effects (font (size 1 1) (thickness 0.15)))
+    )
+    (fp_circle (center 0 0) (end 2.5 0) (layer F.CrtYd) (width 0.05))
+    (fp_circle (center 0 0) (end 2.25 0) (layer Cmts.User) (width 0.15))
+    (fp_text user %R (at 0.3 0) (layer F.Fab)
+      (effects (font (size 1 1) (thickness 0.15)))
+    )
+    (pad 1 thru_hole circle (at 0 0) (size 4.5 4.5) (drill 2.7) (layers *.Cu *.Mask))
+  )
+  (module MountingHole:MountingHole_2.7mm_M2.5_ISO7380_Pad (layer F.Cu)
+    (at 98.75 121.58)
+    (descr "Mounting Hole 2.7mm, M2.5, ISO7380")
+    (tags "mounting hole 2.7mm m2.5 iso7380")
+    (attr virtual)
+    (fp_text reference "" (at 0 -3.7) (layer F.SilkS)
+      (effects (font (size 1 1) (thickness 0.15)))
+    )
+    (fp_text value "" (at 0 3.7) (layer F.Fab) hide
+      (effects (font (size 1 1) (thickness 0.15)))
+    )
+    (fp_circle (center 0 0) (end 2.5 0) (layer F.CrtYd) (width 0.05))
+    (fp_circle (center 0 0) (end 2.25 0) (layer Cmts.User) (width 0.15))
+    (fp_text user %R (at 0.3 0) (layer F.Fab)
+      (effects (font (size 1 1) (thickness 0.15)))
+    )
+    (pad 1 thru_hole circle (at 0 0) (size 4.5 4.5) (drill 2.7) (layers *.Cu *.Mask))
+  )
+  (module MountingHole:MountingHole_2.7mm_M2.5_ISO7380_Pad (layer F.Cu)
+    (at 98.75 72.58)
+    (descr "Mounting Hole 2.7mm, M2.5, ISO7380")
+    (tags "mounting hole 2.7mm m2.5 iso7380")
+    (attr virtual)
+    (fp_text reference "" (at 0 -3.7) (layer F.SilkS)
+      (effects (font (size 1 1) (thickness 0.15)))
+    )
+    (fp_text value "" (at 0 3.7) (layer F.Fab) hide
+      (effects (font (size 1 1) (thickness 0.15)))
+    )
+    (fp_circle (center 0 0) (end 2.5 0) (layer F.CrtYd) (width 0.05))
+    (fp_circle (center 0 0) (end 2.25 0) (layer Cmts.User) (width 0.15))
+    (fp_text user %R (at 0.3 0) (layer F.Fab)
+      (effects (font (size 1 1) (thickness 0.15)))
+    )
+    (pad 1 thru_hole circle (at 0 0) (size 4.5 4.5) (drill 2.7) (layers *.Cu *.Mask))
+  )
+  (module MountingHole:MountingHole_2.7mm_M2.5_ISO7380_Pad (layer F.Cu)
+    (at 156.75 72.58)
+    (descr "Mounting Hole 2.7mm, M2.5, ISO7380")
+    (tags "mounting hole 2.7mm m2.5 iso7380")
+    (attr virtual)
+    (fp_text reference "" (at 0 -3.7) (layer F.SilkS)
+      (effects (font (size 1 1) (thickness 0.15)))
+    )
+    (fp_text value "" (at 0 3.7) (layer F.Fab) hide
+      (effects (font (size 1 1) (thickness 0.15)))
+    )
+    (fp_circle (center 0 0) (end 2.5 0) (layer F.CrtYd) (width 0.05))
+    (fp_circle (center 0 0) (end 2.25 0) (layer Cmts.User) (width 0.15))
+    (fp_text user %R (at 0.3 0) (layer F.Fab)
+      (effects (font (size 1 1) (thickness 0.15)))
+    )
+    (pad 1 thru_hole circle (at 0 0) (size 4.5 4.5) (drill 2.7) (layers *.Cu *.Mask))
   )
   (module Resistor_THT:R_Axial_DIN0207_L6.3mm_D2.5mm_P2.54mm_Vertical (layer F.Cu)
@@
     )
   )
-  (module cidco:MountingHole_2.7mm_M2.5_Pad (layer F.Cu)
-    (at 98.75 121.58)
-    (descr "Mounting Hole 2.7mm, M2.5")
-    (tags "mounting hole 2.7mm m2.5")
-    (attr virtual)
-    (fp_text reference "" (at 0 -3.7) (layer F.SilkS)
-      (effects (font (size 1 1) (thickness 0.15)))
-    )
-    (fp_text value "" (at 0 3.7) (layer F.Fab) hide
-      (effects (font (size 1 1) (thickness 0.15)))
-    )
-    (fp_text user %R (at 0.3 0) (layer F.Fab)
-      (effects (font (size 1 1) (thickness 0.15)))
-    )
-    (fp_circle (center 0 0) (end 2.7 0) (layer Cmts.User) (width 0.15))
-    (fp_circle (center 0 0) (end 2.95 0) (layer F.CrtYd) (width 0.05))
-    (pad "" np_thru_hole circle (at 0 0) (size 2.75 2.75) (drill 2.75) (layers *.Cu *.Mask)
-      (solder_mask_margin 1.725) (clearance 1.725))
-  )
-  (module cidco:MountingHole_2.7mm_M2.5_Pad (layer F.Cu)
-    (at 156.75 121.58)
-    (descr "Mounting Hole 2.7mm, M2.5")
-    (tags "mounting hole 2.7mm m2.5")
-    (attr virtual)
-    (fp_text reference "" (at 0 -3.7) (layer F.SilkS)
-      (effects (font (size 1 1) (thickness 0.15)))
-    )
-    (fp_text value "" (at 0 3.7) (layer F.Fab) hide
-      (effects (font (size 1 1) (thickness 0.15)))
-    )
-    (fp_text user %R (at 0.3 0) (layer F.Fab)
-      (effects (font (size 1 1) (thickness 0.15)))
-    )
-    (fp_circle (center 0 0) (end 2.7 0) (layer Cmts.User) (width 0.15))
-    (fp_circle (center 0 0) (end 2.95 0) (layer F.CrtYd) (width 0.05))
-    (pad "" np_thru_hole circle (at 0 0) (size 2.75 2.75) (drill 2.75) (layers *.Cu *.Mask)
-      (solder_mask_margin 1.725) (clearance 1.725))
-  )
-  (module cidco:MountingHole_2.7mm_M2.5_Pad (layer F.Cu)
-    (at 156.75 72.58)
-    (descr "Mounting Hole 2.7mm, M2.5")
-    (tags "mounting hole 2.7mm m2.5")
-    (attr virtual)
-    (fp_text reference "" (at 0 -3.7) (layer F.SilkS)
-      (effects (font (size 1 1) (thickness 0.15)))
-    )
-    (fp_text value "" (at 0 3.7) (layer F.Fab) hide
-      (effects (font (size 1 1) (thickness 0.15)))
-    )
-    (fp_text user %R (at 0.3 0) (layer F.Fab)
-      (effects (font (size 1 1) (thickness 0.15)))
-    )
-    (fp_circle (center 0 0) (end 2.7 0) (layer Cmts.User) (width 0.15))
-    (fp_circle (center 0 0) (end 2.95 0) (layer F.CrtYd) (width 0.05))
-    (pad "" np_thru_hole circle (at 0 0) (size 2.75 2.75) (drill 2.75) (layers *.Cu *.Mask)
-      (solder_mask_margin 1.725) (clearance 1.725))
-  )
-  (module cidco:MountingHole_2.7mm_M2.5_Pad (layer F.Cu)
-    (at 98.75 72.58)
-    (descr "Mounting Hole 2.7mm, M2.5")
-    (tags "mounting hole 2.7mm m2.5")
-    (attr virtual)
-    (fp_text reference "" (at 0 -3.7) (layer F.SilkS)
-      (effects (font (size 1 1) (thickness 0.15)))
-    )
-    (fp_text value "" (at 0 3.7) (layer F.Fab) hide
-      (effects (font (size 1 1) (thickness 0.15)))
-    )
-    (fp_text user %R (at 0.3 0) (layer F.Fab)
-      (effects (font (size 1 1) (thickness 0.15)))
-    )
-    (fp_circle (center 0 0) (end 2.7 0) (layer Cmts.User) (width 0.15))
-    (fp_circle (center 0 0) (end 2.95 0) (layer F.CrtYd) (width 0.05))
-    (pad "" np_thru_hole circle (at 0 0) (size 2.75 2.75) (drill 2.75) (layers *.Cu *.Mask)
-      (solder_mask_margin 1.725) (clearance 1.725))
-  )
   (module cidco:Pin_Header_Straight_2x20 (layer F.Cu)
